File: MRCS-Adapter-RJ11.sch (EAGLE design)
At the start: 24 parts, among them J10 RJ11, J12 RJ11, J2 RJ11, J4 RJ11, J6 RJ11, J8 RJ11, M1 MOUNTINGHOLE, M10 MOUNTINGHOLE, M11 MOUNTINGHOLE, M12 MOUNTINGHOLE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

Commit message: added missing values
Parts:
- J1, J11, J3, J5, J7, J9: value (none) -> 0.100
- J10, J12, J2, J4, J6, J8: value RJ11 -> 4P4C
Changed lines of the file:
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@@
 <setting verticaltext="up"/>
 </settings>
-<grid distance="0.1" unitdist="inch" unit="inch" style="lines" multiple="1" display="no" altdistance="0.01" altunitdist="inch" altunit="inch"/>
+<grid distance="100" unitdist="mil" unit="mil" style="dots" multiple="1" display="yes" altdistance="50" altunitdist="mil" altunit="mil"/>
 <layers>
 <layer number="1" name="Top" color="4" fill="1" visible="no" active="no"/>
@@
 </classes>
 <parts>
-<part name="J1" library="SPCoast" deviceset="CONNECTOR-M04" device="LOCK"/>
-<part name="J2" library="con-rj" deviceset="RJ11" device=""/>
-<part name="J3" library="SPCoast" deviceset="CONNECTOR-M04" device="LOCK"/>
-<part name="J4" library="con-rj" deviceset="RJ11" device=""/>
-<part name="J5" library="SPCoast" deviceset="CONNECTOR-M04" device="LOCK"/>
-<part name="J6" library="con-rj" deviceset="RJ11" device=""/>
+<part name="J1" library="SPCoast" deviceset="CONNECTOR-M04" device="LOCK" value="0.100"/>
+<part name="J2" library="con-rj" deviceset="RJ11" device="" value="4P4C"/>
+<part name="J3" library="SPCoast" deviceset="CONNECTOR-M04" device="LOCK" value="0.100"/>
+<part name="J4" library="con-rj" deviceset="RJ11" device="" value="4P4C"/>
+<part name="J5" library="SPCoast" deviceset="CONNECTOR-M04" device="LOCK" value="0.100"/>
+<part name="J6" library="con-rj" deviceset="RJ11" device="" value="4P4C"/>
 <part name="FRAME1" library="frames" deviceset="FRAME_A_L" device=""/>
-<part name="J7" library="SPCoast" deviceset="CONNECTOR-M04" device="LOCK"/>
-<part name="J8" library="con-rj" deviceset="RJ11" device=""/>
-<part name="J9" library="SPCoast" deviceset="CONNECTOR-M04" device="LOCK"/>
-<part name="J10" library="con-rj" deviceset="RJ11" device=""/>
-<part name="J11" library="SPCoast" deviceset="CONNECTOR-M04" device="LOCK"/>
-<part name="J12" library="con-rj" deviceset="RJ11" device=""/>
+<part name="J7" library="SPCoast" deviceset="CONNECTOR-M04" device="LOCK" value="0.100"/>
+<part name="J8" library="con-rj" deviceset="RJ11" device="" value="4P4C"/>
+<part name="J9" library="SPCoast" deviceset="CONNECTOR-M04" device="LOCK" value="0.100"/>
+<part name="J10" library="con-rj" deviceset="RJ11" device="" value="4P4C"/>
+<part name="J11" library="SPCoast" deviceset="CONNECTOR-M04" device="LOCK" value="0.100"/>
+<part name="J12" library="con-rj" deviceset="RJ11" device="" value="4P4C"/>
 <part name="M1" library="SPCoast" deviceset="MOUNTINGHOLE" device=""/>
 <part name="M2" library="SPCoast" deviceset="MOUNTINGHOLE" device=""/>
