File: MRCS-Adapter-RJ11.brd (EAGLE design)
At the start: 128.3 x 106.7 mm, 31 parts, among them J10 RJ11, J12 RJ11, J2 RJ11, J4 RJ11, J6 RJ11, J8 RJ11, M1 MOUNTINGHOLE, M10 MOUNTINGHOLE, M11 MOUNTINGHOLE, M12 MOUNTINGHOLE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

Commit message: added missing values
Parts:
- J1, J11, J3, J5, J7, J9: value (none) -> 0.100
- J10, J12, J2, J4, J6, J8: value RJ11 -> 4P4C
- U$1, U$2, U$3, U$4, U$5, U$6: value (none) -> MRCS
Changed lines of the file:
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@@
 <setting verticaltext="up"/>
 </settings>
-<grid distance="1" unitdist="mm" unit="mm" style="lines" multiple="1" display="no" altdistance="0.025" altunitdist="inch" altunit="mil"/>
+<grid distance="50" unitdist="mil" unit="mil" style="dots" multiple="2" display="yes" altdistance="25" altunitdist="mil" altunit="mil"/>
 <layers>
 <layer number="1" name="Top" color="4" fill="1" visible="yes" active="yes"/>
@@
 <elements>
 <element name="E$1" library="SPCoast" package="BOARD-10X10-3X2-PANEL" value="" x="0" y="0"/>
-<element name="J1" library="SPCoast" package="1X04_LOCK" value="" x="5.08" y="44.45" rot="R90"/>
-<element name="J2" library="con-rj" package="RJ11" value="RJ11" x="39.37" y="49.53"/>
-<element name="U$1" library="MRCSLogoTop" package="MRCSLOGOTOP" value="" x="5.08" y="57.15"/>
-<element name="J3" library="SPCoast" package="1X04_LOCK" value="" x="5.08" y="73.12" rot="R90"/>
-<element name="J4" library="con-rj" package="RJ11" value="RJ11" x="39.37" y="78.2"/>
-<element name="J5" library="SPCoast" package="1X04_LOCK" value="" x="5.08" y="16.51" rot="R90"/>
-<element name="J6" library="con-rj" package="RJ11" value="RJ11" x="39.37" y="21.59"/>
-<element name="J7" library="SPCoast" package="1X04_LOCK" value="" x="54.61" y="16.51" rot="R90"/>
-<element name="J8" library="con-rj" package="RJ11" value="RJ11" x="88.9" y="21.59"/>
-<element name="J9" library="SPCoast" package="1X04_LOCK" value="" x="54.61" y="73.12" rot="R90"/>
-<element name="J10" library="con-rj" package="RJ11" value="RJ11" x="88.9" y="78.2"/>
-<element name="J11" library="SPCoast" package="1X04_LOCK" value="" x="54.61" y="44.45" rot="R90"/>
-<element name="J12" library="con-rj" package="RJ11" value="RJ11" x="88.9" y="49.53"/>
-<element name="U$2" library="MRCSLogoTop" package="MRCSLOGOTOP" value="" x="52.07" y="57.15"/>
-<element name="U$3" library="MRCSLogoTop" package="MRCSLOGOTOP" value="" x="5.08" y="29.21"/>
-<element name="U$4" library="MRCSLogoTop" package="MRCSLOGOTOP" value="" x="53.34" y="29.21"/>
-<element name="U$5" library="MRCSLogoTop" package="MRCSLOGOTOP" value="" x="5.08" y="85.09"/>
-<element name="U$6" library="MRCSLogoTop" package="MRCSLOGOTOP" value="" x="53.34" y="85.09"/>
+<element name="J1" library="SPCoast" package="1X04_LOCK" value="0.100" x="5.08" y="44.45" rot="R90"/>
+<element name="J2" library="con-rj" package="RJ11" value="4P4C" x="39.37" y="49.53"/>
+<element name="U$1" library="MRCSLogoTop" package="MRCSLOGOTOP" value="MRCS" x="5.08" y="57.15"/>
+<element name="J3" library="SPCoast" package="1X04_LOCK" value="0.100" x="5.08" y="73.12" rot="R90"/>
+<element name="J4" library="con-rj" package="RJ11" value="4P4C" x="39.37" y="78.2"/>
+<element name="J5" library="SPCoast" package="1X04_LOCK" value="0.100" x="5.08" y="16.51" rot="R90"/>
+<element name="J6" library="con-rj" package="RJ11" value="4P4C" x="39.37" y="21.59"/>
+<element name="J7" library="SPCoast" package="1X04_LOCK" value="0.100" x="54.61" y="16.51" rot="R90"/>
+<element name="J8" library="con-rj" package="RJ11" value="4P4C" x="88.9" y="21.59"/>
+<element name="J9" library="SPCoast" package="1X04_LOCK" value="0.100" x="54.61" y="73.12" rot="R90"/>
+<element name="J10" library="con-rj" package="RJ11" value="4P4C" x="88.9" y="78.2"/>
+<element name="J11" library="SPCoast" package="1X04_LOCK" value="0.100" x="54.61" y="44.45" rot="R90"/>
+<element name="J12" library="con-rj" package="RJ11" value="4P4C" x="88.9" y="49.53"/>
+<element name="U$2" library="MRCSLogoTop" package="MRCSLOGOTOP" value="MRCS" x="52.07" y="57.15"/>
+<element name="U$3" library="MRCSLogoTop" package="MRCSLOGOTOP" value="MRCS" x="5.08" y="29.21"/>
+<element name="U$4" library="MRCSLogoTop" package="MRCSLOGOTOP" value="MRCS" x="53.34" y="29.21"/>
+<element name="U$5" library="MRCSLogoTop" package="MRCSLOGOTOP" value="MRCS" x="5.08" y="85.09"/>
+<element name="U$6" library="MRCSLogoTop" package="MRCSLOGOTOP" value="MRCS" x="53.34" y="85.09"/>
 <element name="M1" library="SPCoast" package="MOUNTINGHOLE" value="MOUNTINGHOLE" x="20.32" y="12.065"/>
 <element name="M2" library="SPCoast" package="MOUNTINGHOLE" value="MOUNTINGHOLE" x="20.32" y="30.48"/>

Commit message: added missing values
Parts:
- E$1: value (none) -> 10x10
Changed lines of the file:
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@@
 </autorouter>
 <elements>
-<element name="E$1" library="SPCoast" package="BOARD-10X10-3X2-PANEL" value="" x="0" y="0"/>
+<element name="E$1" library="SPCoast" package="BOARD-10X10-3X2-PANEL" value="10x10" x="0" y="0"/>
 <element name="J1" library="SPCoast" package="1X04_LOCK" value="0.100" x="5.08" y="44.45" rot="R90"/>
 <element name="J2" library="con-rj" package="RJ11" value="4P4C" x="39.37" y="49.53"/>
